File: BeagleBone_Black_Wireless.brd (EAGLE design)
At the start: 86.4 x 54.6 mm, 277 parts, among them IC1 OSD3358, IC10 TXS0108ERGYR, IC11 TXS0108ERGYR, IC12 TPS2051BDGN, IC13 SN74AUC1G74, IC14 TPD4S012DRY, IC15 TPD4S012DRY, IC16 AM29F040E, IC17 SN74LVC2G241DCUR, IC18 TL1963ADCQR, IC19 AP2112K-1.8TRG1 3.3V, IC2 SN74LVC1G07DCK, IC20 AM29F040E, IC3 SN74LVC1G06DCK, IC4 24LC32AT-I/OT, IC5 TLVH431 (SOT-23-3), IC6 DNP TLVH431 (SOT-23-3), IC7 IP4283CZ10-TBR, IC8 IP4283CZ10-TBR, IC9 TDA19988BHN/C1,557, Q2 32.768kHz, Q4 24 MHz, T1 MMBT2907, T2 DNP MMBT2907, T3 BSS138W-7-F, T4 BSS138W-7-F, X2 SCHA5B0200, X4 10118192-0001LF, X5 10118241-001RLF

Commit message: changes 2
Parts:
- removed C27, C28, C29, C30, C31, C32, C33, C34, C35, C36, C37, C38, C39, C40, C41, C42: 47pF, 6.3V, rcl:C0402K
- removed C50, C51, C52, C53, C59: .1uF, 6.3V, rcl:C0402K
- removed C54, C55, C56, C57: 2.2uF, 6.3V, rcl:C0603K
- removed D1: RB751V40,115, GHI-BasicComponents:SOD323(NXP)REFLOW
- removed F1: 1206L025YR, inductor-neosid:SM-1206
- removed FB2: 2.5k Ohm (BLM18BD252SN1D), GHI-BasicComponents:0805-RESISTOR
- removed IC14: TPD4S012DRY, GHI-IC:SON-6(TI)-DRY
- removed IC16: AM29F040E, am29-memory:TSOP32
- removed R114: 0, 1%, rcl:R0402
- removed R115, R118: 1.5k, 1%, rcl:R0402
- removed R119, R121: 10k, 1%, rcl:R0402
- removed R120: 27k, 1%, rcl:R0402
- removed X4: 10118192-0001LF, GHI-Connectors:10118192-0001LF(MICRO-USB-B-AMPHENOL-FCI)
- removed X5: 10118241-001RLF, GHI-Connectors:HDMI-TYPE-D-10118241
- IC7, IC8: value IP4283CZ10-TBR -> 75162P; device GHI-IC:SOT1176-1(NXP) -> 751xx:DIL22-3
- IC9: value TDA19988BHN/C1,557 -> 75162P; device GHI-IC:SOT804-4(NXP) -> 751xx:DIL22-3
- moved IC9 113.5 mm to (-10.0, -40.2), turned to 0 degrees
- moved IC8 95.5 mm to (-10.0, -28.1), flipped to the top, turned to 0 degrees
- moved IC7 87.8 mm to (-10.0, -16.0), flipped to the top, turned to 0 degrees
Connections:
- removed net CEC: D1.C, IC9.30, X5.15
- removed net DVI_5V: F1.1, R115.1, R118.1, X5.19
- removed net EXT_SWING: IC9.34, R119.1
- removed net HDMI.DSCL: IC9.33, R115.2, X5.17
- removed net HDMI.DSDA: IC9.32, R118.2, X5.18
- removed net HDMI_1V8: C50.1, C51.1, C52.1, C53.1, C54.1, C55.1, C56.1, C57.1, FB2.2, IC9.14, IC9.29, IC9.35, IC9.36, IC9.41, IC9.46, IC9.47, IC9.48, IC9.5, IC9.55
- removed net HPD: IC9.31, X5.1
- removed net N$10: IC20.1, IC20.10, IC20.11, IC20.12, IC20.13, IC20.2, IC20.3, IC20.30, IC20.31, IC20.32, IC20.4, IC20.5, IC20.6, IC20.7, IC20.9
- removed net N$21: IC16.7, IC20.29
- removed net N$23: IC16.32, IC20.28
- removed net N$26: IC16.30, IC20.27
- removed net TEST: IC9.49, R114.2
- removed net TX0+: IC8.5, IC9.40, X5.9
- removed net TX0-: IC8.4, IC9.39, X5.11
- removed net TX1+: IC7.2, IC9.43, X5.6
- removed net TX1-: IC7.1, IC9.42, X5.8
- removed net TX2+: IC7.5, IC9.45, X5.3
- removed net TX2-: IC7.4, IC9.44, X5.5
- removed net TXC+: IC8.2, IC9.38, X5.12
- removed net TXC-: IC8.1, IC9.37, X5.14
- new net N$55: IC7.12, IC8.9
- new net N$60: IC7.2, IC8.8
- new net N$61: IC7.1, IC7.13, IC7.14, IC7.15, IC8.10
- net 12MHZ: no longer IC9.27
- net CGND: no longer X4.CGND1, X4.CGND2, X4.CGND3, X4.CGND4, X4.CGND5, X4.CGND6, X5.CG1, X5.CG2, X5.CG3, X5.CG4
- net GND: now also IC7.11, IC8.11, IC9.11; no longer C27.2, C28.2, C29.2, C30.2, C31.2, C32.2, C33.2, C34.2, C35.2, C36.2, C37.2, C38.2, C39.2, C40.2, C41.2, C42.2, C50.2, C51.2, C52.2, C53.2, C54.2, C55.2, C56.2, C57.2, C59.2, IC14.4, IC16.24, IC4.2, IC7.3, IC7.8, IC8.3, IC8.8, IC9.16, IC9.17, IC9.18, IC9.19, IC9.53, IC9.54, IC9.61, IC9.62, IC9.63, IC9.65, IC9.8, IC9.9, R114.1, R119.2, X4.GND, X5.10, X5.13, X5.16, X5.4, X5.7
- net HDMICLK_DIS#: now also R104.2
- net HDMI_INT: no longer IC9.50, R121.2
- net I2C0_SCL: now also IC1.R8; no longer IC9.52
- net I2C0_SDA: now also IC1.U8; no longer IC9.51
- net LCD.CLOCK: no longer IC9.4
- net LCD.D0.B0--B3: no longer C42.1, IC9.15
- net LCD.D1.B1--B4: no longer C41.1, IC9.13
- net LCD.D10.G5--G7: no longer C32.1, IC9.64
- net LCD.D11.R0--R3: no longer C31.1, IC9.60
- net LCD.D12.R1--R4: no longer C30.1, IC9.59
- net LCD.D13.R2--R5: no longer C29.1, IC9.58
- net LCD.D14.R3--R6: no longer C28.1, IC9.57
- net LCD.D15.R4--R7: no longer C27.1, IC9.56
- net LCD.D2.B2--B5: no longer C40.1, IC9.12
- net LCD.D3.B3--B6: no longer C39.1, IC9.11
- net LCD.D4.B4--B7: no longer C38.1, IC9.10
- net LCD.D5.G0--G2: no longer C37.1, IC9.7
- net LCD.D6.G1--G3: no longer C36.1, IC9.6
- net LCD.D7.G2--G4: no longer C35.1, IC9.3
- net LCD.D8.G3--G5: no longer C34.1, IC9.2
- net LCD.D9.G4--G6: no longer C33.1, IC9.1
- net LCD.ENABLE: no longer IC9.20
- net LCD.HSYNC: no longer IC9.22
- net LCD.VSYNC: no longer IC9.21
- net MMC1_DAT2: no longer IC1.R8
- net MMC1_DAT3: now also IC4.2
- net MMC1_DAT4: no longer IC1.U8
- net N$27: now also IC20.29; no longer IC16.20
- net N$32: now also IC20.28; no longer IC16.19
- net N$46: now also IC20.27; no longer IC16.18
- net N$66: now also IC7.16, IC7.17, IC7.18, IC7.19, IC7.20, IC8.3; no longer D1.A, R120.2
- net SPI1_CS0: no longer IC9.25
- net SPI1_D0: no longer IC9.24
- net SPI1_SCLK: no longer IC9.23
- net SYS_5V: no longer F1.2
- net USB.CLIENT.D+: no longer IC14.1, X4.D+
- net USB.CLIENT.D-: no longer IC14.2, X4.D-
- net USB.CLIENT.ID: no longer IC14.3, X4.ID
- net USB_DC: no longer C59.1, IC14.6, X4.VBUS
- net USR0: no longer R104.2
- net VCC: now also IC7.22, IC8.22, IC9.22; no longer IC16.8
- net VDD_1V8: no longer FB2.1
- net VDD_3V3B: no longer R120.1, R121.1
Routing:
- net HDMI_1V8: track 80.7 -> 0.00 mm, vias 8 -> 0
- net GND: track 254.4 -> 196.7 mm, vias 96 -> 79
- net LCD.D14.R3--R6: track 41.5 -> 4.60 mm, vias 3 -> 2
- net USR0: track 35.0 -> 1.08 mm, vias 2 -> 1
- net HDMICLK_DIS#: track 20.8 -> 54.7 mm, vias 2 -> 3
- net LCD.D11.R0--R3: track 44.0 -> 10.2 mm, vias 3 -> 2
- net TX1-: track 32.9 -> 0.00 mm, vias 2 -> 0
- net LCD.D13.R2--R5: track 46.0 -> 13.2 mm, vias 2 -> 1
- net USB.CLIENT.D+: track 40.8 -> 9.02 mm, vias 2 -> 1
- net TX1+: track 31.3 -> 0.00 mm, vias 2 -> 0
- net USB.CLIENT.ID: track 41.3 -> 10.9 mm, vias 2 -> 1
- net TXC+: track 29.6 -> 0.00 mm, vias 2 -> 0
- net TX2+: track 27.4 -> 0.00 mm, vias 1 -> 0
- net TXC-: track 27.2 -> 0.00 mm, vias 2 -> 0
- net TX2-: track 26.7 -> 0.00 mm, vias 1 -> 0
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